File: MAX31865.kicad_pcb (KiCad board)
At the start: 2 copper layers, 25.4 x 27.9 mm, 29 parts, among them U1 MAX31865, U3 MIC5225-3.3, X1 3.5mm, X2 3.5mm

Commit message: temp
Parts:
- removed U$16: , ADAFRUIT_3.5MM
- removed U$20, U$21: , ADAFRUIT_5MM
- removed U$8: , PCBFEAT-REV-040
- FB1: value (none) -> FERRITE-0805NO
- J1: renamed from JP1; value (none) -> HEADER-1X870MIL; moved to B.Cu
- SJ1: value (none) -> SOLDERJUMPER_2WAY
- SJ3, SJ4: value (none) -> SOLDERJUMPER
- moved J1 17.6 mm to (157.5, 116.3)
- moved X1 4.24 mm to (149.8, 94.5), turned to 0 degrees
- moved X2 4.23 mm to (142.8, 94.6), turned to 0 degrees
- moved FID1 0.56 mm to (159.3, 97.8)
- moved U2 0.16 mm to (140.3, 109.6)
- moved C4 0.07 mm to (140.3, 113.0)
- turned SJ1 to 180 degrees
- renumbered U3 to U2
Connections:
- net FORCE- renamed Net-(SJ4-A)
- net RTDIN+ renamed Net-(SJ3-A)
- net RTDIN- renamed Net-(SJ4-B)
- D1 pad 1: (no net) -> /SDI_5V
- D1 pad 2: (no net) -> Net-(D1-A)
- D2 pad 1: (no net) -> /SCLK_5V
- D2 pad 2: (no net) -> Net-(D2-A)
- D3 pad 1: (no net) -> /CS_5V
- D3 pad 2: (no net) -> Net-(D3-A)
- J1 pad 1: VIN -> /DRDY
- J1 pad 2: GND -> /CS_5V
- J1 pad 3: VDD -> /SDI_5V
- J1 pad 4: SCLK_5V -> /SDO
- J1 pad 5: SDO -> /SCLK_5V
- J1 pad 6: SDI_5V -> VDD
- J1 pad 7: CS_5V -> GND
- J1 pad 8: DRDY -> VIN
- R6 pad 1: N$14 -> /DRDY
- R7 pad 1: N$12 -> Net-(D3-A)
- R8 pad 1: N$13 -> Net-(D2-A)
- SJ1 pad 1: GND -> Net-(SJ1-A)
- SJ1 pad 3: FORCE+ -> GND
- SJ3 pad 2: FORCE+ -> Net-(SJ1-A)
- U1 pad 11: N$14 -> Net-(D1-A)
- U1 pad 12: N$13 -> Net-(D2-A)
- U1 pad 13: N$12 -> Net-(D3-A)
- U1 pad 14: SDO -> /SDO
- U1 pad 17: (no net) -> unconnected-(U1-NC-Pad17)
- U1 pad 18: DRDY -> /DRDY
- U1 pad 5: FORCE+ -> Net-(SJ1-A)
- U2 pad 4: (no net) -> unconnected-(U2-P4-Pad4)
- X1 pad 2: FORCE+ -> Net-(SJ1-A)
Routing:
- net N$14: track 21.5 -> 0.00 mm, vias 2 -> 0
- net /DRDY: track 0.00 -> 21.4 mm, vias 0 -> 2
- net Net-(D3-A): track 0.00 -> 21.4 mm, vias 0 -> 2
- net N$12: track 21.4 -> 0.00 mm, vias 2 -> 0
- net DRDY: track 19.4 -> 0.00 mm, vias 1 -> 0
- net SDO: track 18.8 -> 0.00 mm, vias 1 -> 0
- net Net-(D1-A): track 0.00 -> 18.7 mm, vias 0 -> 2
- net /SDO: track 0.00 -> 18.7 mm, vias 0 -> 1
- net Net-(SJ1-A): track 0.00 -> 17.5 mm
- net FORCE+: track 17.0 -> 0.00 mm
- net Net-(D2-A): track 0.00 -> 12.0 mm
- net N$13: track 11.6 -> 0.00 mm
- net GND: track 8.61 -> 13.8 mm, vias 5 -> 7
- net CS_5V: track 3.55 -> 0.00 mm
- net /CS_5V: track 0.00 -> 3.55 mm
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Other:
- board text removed: "2 Wire"
- board text removed: "2/3 Wire"
- board text removed: "2/3/4 Wire Platinum RTD Converter"
- board text removed: "24"
- board text removed: "3"
- board text removed: "F+"
- board text removed: "F-"
- board text removed: "MAX31865"
- board text removed: "RTD+"
- board text removed: "RTD-"
- board text removed: "Vin: 3-5VDC Vlogic: 3-5VDC"
