File: MAX31865.kicad_sch (KiCad schematic)
At the start: 25 parts, among them U1 MAX31865, U2 MIC5225-3.3, X1 3.5mm, X2 3.5mm

Commit message: temp
Parts:
- removed FID1, FID2: FIDUCIAL{dblquote}{dblquote}, Fiducial:Fiducial_1mm_Mask2mm, symbol MAX31865-eagle-import:FIDUCIAL{dblquote}{dblquote}
- C1, C2, C3: symbol Device:C -> Device:C_Small
- C4, C5: symbol Device:C -> Device:C_Small; Component package type (none) -> C_0805; MPN (none) -> /; Manufacturer (none) -> /; SPN (none) -> GPC0805106-16; Supplier (none) -> Eurocircuits
- D1, D2, D3: Component package type (none) -> SOD-323; MPN (none) -> 1N4148WX-TP; Manufacturer (none) -> Micro Commercial Co; SPN (none) -> 1N4148WXTPMSTR-ND; Supplier (none) -> DigiKey
- FB1: symbol Device:FerriteBead -> Device:FerriteBead_Small
- J1: renamed from JP1; value HEADER-1X870MIL -> <; footprint Connector_PinHeader_1.00mm:PinHeader_1x08_P1.00mm_Vertical -> Connector_PinHeader_2.54mm:PinHeader_1x08_P2.54mm_Vertical; Component package type (none) -> /; MPN (none) -> TSW-108-09-G-S; Manufacturer (none) -> Samtec Inc.; SPN (none) -> SAM12332-ND; Supplier (none) -> DigiKey
- R1: symbol Device:R -> Device:R_Small
- U$18, U$19: symbol MAX31865-eagle-import:MOUNTINGHOLE2.5 -> Mechanical:MountingHole; now left out of the parts list
- U2: Component package type (none) -> SOT-235; MPN (none) -> MIC5225-3.3YM5-TR; Manufacturer (none) -> Microchip Technology; SPN (none) -> 576-2980-2-ND; Supplier (none) -> DigiKey
Connections:
- no-connect marks 0 -> 1
Other:
- moved on the sheet: C1, C2, C3, C4, C5, D1, D2, D3, FB1, J1, R1, R6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
