File: MAX31865.kicad_sch (KiCad schematic)
At the start: 22 parts, among them J1 connector, J2 Screw_Terminal_01x04, U1 MAX31865, U2 MIC5225

Commit message: docs: fill in the title block
Other:
- company: (none) -> UHasselt, Solar Cooker
Changed lines of the file:
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@@
 	(title_block
 		(title "MAX31865")
-		(date "2024-03-06")
+		(date "2026-10-18")
+		(rev "1.0")
+		(company "UHasselt, Solar Cooker")
+		(comment 1 "Based on the Adafruit MAX31865 RTD amplifier breakout")
+		(comment 2 "Design: Lowie Van Vyve")
+		(comment 3 "github.com/solar-cooker-UHasselt/kicad-adafruit-max31865")
 	)
 	(text "JP1 to GND for 2/4-wire, to FORCE+ for 3-wire"
